Commit message: Third commit of ASIMOV workspace

File: arm_urdf/urdf/arm_urdf.urdf (robot description, URDF)
Before this commit: robot arm_urdf, 7 links, 6 joints
Joints:
- joint joint_1: limit (none) -> lower=-1.5708 upper=1.5708 effort=200 velocity=3; type continuous -> revolute
- joint joint_2: limit (none) -> lower=0.3491 upper=2.5307 effort=200 velocity=3; type continuous -> revolute
- joint joint_3: limit (none) -> lower=0 upper=2.4435 effort=200 velocity=3; type continuous -> revolute
- joint joint_4: limit (none) -> lower=-1.309 upper=1.309 effort=200 velocity=3; type continuous -> revolute
- joint left_claw_joint: type continuous -> revolute
- joint right_claw_joint: type continuous -> revolute

Commit message: First Working Prototype of Arm Control

File: arm_urdf/urdf/arm_urdf.urdf (robot description, URDF)
Before this commit: robot arm_urdf, 7 links, 6 joints
Joints:
- joint joint_1: limit lower=-1.5708 upper=1.5708 effort=200 velocity=3 -> (none); type revolute -> continuous
- joint joint_2: limit lower=0.3491 upper=2.5307 effort=200 velocity=3 -> (none); type revolute -> continuous
- joint joint_3: limit lower=0 upper=2.4435 effort=200 velocity=3 -> (none); type revolute -> continuous
- joint joint_4: limit lower=-1.309 upper=1.309 effort=200 velocity=3 -> (none); type revolute -> continuous
- joint left_claw_joint: type revolute -> continuous
- joint right_claw_joint: type revolute -> continuous
